Commit message: Servos 2 to 6 OK Claw and model not conforming

File: ros2_ws/src/xarm/urdf/xarm_1s.urdf.xacro (robot description, xacro)
@@ -32,6 +32,6 @@
     <parent link="base_link"/>
     <child link="link6"/>
-    <origin rpy="0.0 0.0 0.0" xyz="0.0 0.0 0.043"/>
-    <axis xyz="0 0 1"/>
+    <origin rpy="0.0 0.0 3.14" xyz="0.0 0.0 0.043"/>
+    <axis xyz="0 0 -1"/>
   </joint>
   <link name="link6">
@@ -77,5 +77,5 @@
     <child link="link4"/>
     <origin rpy="0.0 0.0 0.0" xyz="0.0 0.0 0.09775"/>
-    <axis xyz="0 1 0"/>
+    <axis xyz="0 -1 0"/>
   </joint>
   <link name="link4">
